File: Hardware/MPU.kicad_sch (KiCad schematic)
At the start: 18 parts, among them J6 USB_C_Receptacle_USB2.0_16P, U14 AP2112K-3.3, U2 STM32H723VGTx

Commit message: 19-feb update
Parts:
- removed C43, C44, C45, C46, C47, C49: 100nF, Capacitor_SMD:C_0201_0603Metric, symbol Device:C
- removed C48: 4.7uf, Capacitor_SMD:C_0603_1608Metric, symbol Device:C
- removed C50: 1uF, Capacitor_SMD:C_0201_0603Metric, symbol Device:C
- removed D11, D12, D13, D14, D15: BZV55B5V1, Diode_SMD:D_MiniMELF, symbol Diode:BZV55B5V1
- removed J6: USB_C_Receptacle_USB2.0_16P, Connector_USB:USB_C_Receptacle_G-Switch_GT-USB-7010ASV, symbol Connector:USB_C_Receptacle_USB2.0_16P
- removed R21, R22: R, Resistor_SMD:R_01005_0402Metric_Pad0.57x0.30mm_HandSolder, symbol Device:R
- removed U14: AP2112K-3.3, Package_TO_SOT_SMD:SOT-23-5, symbol Regulator_Linear:AP2112K-3.3
- removed U2: STM32H723VGTx, Package_QFP:LQFP-100_14x14mm_P0.5mm, symbol MCU_ST_STM32H7:STM32H723VGTx
- added R25: DNF, Resistor_SMD:R_0603_1608Metric, symbol Device:R
- added R26, R27: 10, Resistor_SMD:R_0201_0603Metric_Pad0.64x0.40mm_HandSolder, symbol Device:R
- added U2: MIMXRT1062DVJ6B, MIMXRT1062DVJ6B:BGA196C80P14X14_1200X1200X152N, symbol MIMXRT1062DVJ6B:MIMXRT1062DVJ6B
Connections:
- net GND: now also R26.2, R27.2
- net MPU-D+: now also U2.L8 (USB_OTG1_DP)
- net MPU-D-: now also U2.M8 (USB_OTG1_DN)
- new net: R25.2, R26.1
- new net DCDC_GND: U2.N1 (DCDC_GND), U2.N2 (DCDC_GND)
- new net DCDC_IN: U2.L1 (DCDC_IN), U2.L2 (DCDC_IN)
- new net DCDC_LP: U2.M1 (DCDC_LP), U2.M2 (DCDC_LP)
- new net MPU-BOOT0: R27.1
- new net MPU-NRST: R25.1
- new net NVCC_EMC: U2.E6 (NVCC_EMC), U2.F5 (NVCC_EMC)
- new net NVCC_GPIO: U2.E9 (NVCC_GPIO), U2.F10 (NVCC_GPIO), U2.J10 (NVCC_GPIO)
- new net VDD_SOC_IN: U2.F6 (VDD_SOC_IN), U2.F7 (VDD_SOC_IN), U2.F8 (VDD_SOC_IN), U2.F9 (VDD_SOC_IN), U2.G6 (VDD_SOC_IN), U2.G9 (VDD_SOC_IN), U2.H6 (VDD_SOC_IN), U2.H9 (VDD_SOC_IN), U2.J9 (VDD_SOC_IN)
- new net VSS: U2.A1 (VSS), U2.A14 (VSS), U2.B10 (VSS), U2.B5 (VSS), U2.E13 (VSS), U2.E2 (VSS), U2.G7 (VSS), U2.G8 (VSS), U2.H7 (VSS), U2.H8 (VSS), U2.J7 (VSS), U2.J8 (VSS), U2.K13 (VSS), U2.K2 (VSS), U2.L9 (VSS), U2.N5 (VSS), U2.N8 (VSS), U2.P1 (VSS), U2.P14 (VSS)

Commit message: 27 feb update
Parts:
- removed R25: DNF, Resistor_SMD:R_0603_1608Metric, symbol Device:R
- removed R26, R27: 10, Resistor_SMD:R_0201_0603Metric_Pad0.64x0.40mm_HandSolder, symbol Device:R
- added D23: LED, LED_SMD:LED_1206_3216Metric_Pad1.42x1.75mm_HandSolder, symbol Device:LED
- added R17: 470, Resistor_SMD:R_0201_0603Metric_Pad0.64x0.40mm_HandSolder, symbol Device:R
Connections:
- net VSS is gone; now on net DCDC_GND: U2.A1 (VSS), U2.A14 (VSS), U2.B10 (VSS), U2.B5 (VSS), U2.E13 (VSS), U2.E2 (VSS), U2.G7 (VSS), U2.G8 (VSS), U2.H7 (VSS), U2.H8 (VSS), U2.J7 (VSS), U2.J8 (VSS), U2.K13 (VSS), U2.K2 (VSS), U2.L9 (VSS), U2.N5 (VSS), U2.N8 (VSS), U2.P1 (VSS), U2.P14 (VSS)
- net DCDC_GND: now also U2.G14 (GPIO_AD_B0_05), R17.1
- net D0: now reaches U2.A12 (GPIO_B1_08)
- net D1: now reaches U2.A13 (GPIO_B1_09)
- net CLK: now reaches U2.B12 (GPIO_B1_07)
- net D2: now reaches U2.B13 (GPIO_B1_10)
- net CS: now reaches U2.C12 (GPIO_B1_06)
- net D3: now reaches U2.C13 (GPIO_B1_11)
- net at U2.D8 (GPIO_B0_03): now also D23.2 (A)
- net PTA6: now reaches U2.E14 (GPIO_AD_B0_06)
- net PTA6: now also U2.G13 (GPIO_AD_B0_10)
- net PTA4: now reaches U2.F11 (GPIO_AD_B0_04)
- net PTB0: now reaches U2.F12 (GPIO_AD_B0_07)
- net PTB5: now reaches U2.F13 (GPIO_AD_B0_08)
- net PTA7: now reaches U2.F14 (GPIO_AD_B0_09)
- net AD_B0_11: now reaches U2.G10 (GPIO_AD_B0_11)
- net PTB4: now reaches U2.L14 (GPIO_AD_B0_13)
- net PTA1: now reaches U2.F3 (GPIO_EMC_01)
- net DCDC_SENSE: now reaches U2.J5 (DCDC_SENSE)
- net NVCC_SD0: now reaches U2.J6 (NVCC_SD0)
- net DCDC_PSWITCH: now reaches U2.K3 (DCDC_PSWITCH)
- net DCDC_IN_Q: now reaches U2.K4 (DCDC_IN_Q)
- net NVCC_SD1: now reaches U2.K5 (NVCC_SD1)
- net PMIC_ON_REQ: now reaches U2.K7 (PMIC_ON_REQ)
- net VDD_USB_CAP: now reaches U2.K8 (VDD_USB_CAP)
- net VDD_SNVS_CAP: now reaches U2.M10 (VDD_SNVS_CAP)
- net PTB1: now reaches U2.M7 (POR_B)
- net VDD_SNVS_IN: now reaches U2.M9 (VDD_SNVS_IN)
- net XTALO: now reaches U2.N11 (XTALO)
- net VDDA_ADC_3P3: now reaches U2.N14 (VDDA_ADC_3P3)
- net USB_OTG1_VBUS: now reaches U2.N6 (USB_OTG1_VBUS)
- net RTC_XTALI: now reaches U2.N9 (RTC_XTALI)
- net NVCC_PLL: now reaches U2.P10 (NVCC_PLL)
- net XTALI: now reaches U2.P11 (XTALI)
- net VDD_HIGH_IN: now reaches U2.P12 (VDD_HIGH_IN)
- net USB_OTG2_VBUS: now reaches U2.P6 (USB_OTG2_VBUS)
- net VDD_HIGH_CAP: now reaches U2.P8 (VDD_HIGH_CAP)
- net RTC_XTALO: now reaches U2.P9 (RTC_XTALO)
- new net: D23.1 (K), R17.2

Commit message: 12-March update
Parts:
- added BZ1: Buzzer, MLT-8530_JHE:MLT-8530_JHE_1, symbol Device:Buzzer
- added D32: WS2812, LED_SMD:LED_WS2812_PLCC6_5.0x5.0mm_P1.6mm, symbol LED:WS2812
- added J9: Conn_01x02, Connector_PinSocket_1.00mm:PinSocket_1x02_P1.00mm_Vertical, symbol Connector_Generic:Conn_01x02
Connections:
- net DCDC_GND: now also BZ1.2 (-), D32.3 (VCC), D32.6 (VSS)
- net MPU-CS: now reaches U2.G11 (GPIO_AD_B0_03)
- net MPI-MOSI: now reaches U2.H10 (GPIO_AD_B0_01)
- net TEL-MPU-MOSI: now reaches U2.J1 (GPIO_SD_B0_02)
- net TEL-MPU-CS: now reaches U2.J3 (GPIO_SD_B0_01)
- net TEL-MPU-SCK: now reaches U2.J4 (GPIO_SD_B0_00)
- net TEL-MPU-MISO: now reaches U2.K1 (GPIO_SD_B0_03)
- net OSD-RESET: now reaches U2.K14 (GPIO_AD_B0_12)
- net NAV-MPU-CS: now reaches U2.L3 (GPIO_SD_B1_06)
- net NAV-MPU-SCK: now reaches U2.L4 (GPIO_SD_B1_07)
- net MPU-MISO: now reaches U2.M11 (GPIO_AD_B0_02)
- net MPU-SCK: now reaches U2.M14 (GPIO_AD_B0_00)
- net NAV-MPU-MISO: now reaches U2.N4 (GPIO_SD_B1_09)
- net NAV-MPU-MOSI: now reaches U2.P3 (GPIO_SD_B1_08)
- net at U2.D3 (GPIO_EMC_24): now also BZ1.1 (+)
- net MPU-stat: now reaches U2.G2 (GPIO_EMC_23)
- net MPU-stat: now also D32.2 (DIN)
- net at U2.N7 (USB_OTG2_DN): now also J9.2 (Pin_2)
- net at U2.P7 (USB_OTG2_DP): now also J9.1 (Pin_1)
- new net 5V-MPU: D32.5 (VDD)
