File: Hardware/Blitz.kicad_pcb (KiCad board)
At the start: 2 copper layers, 108 parts, among them J1 USB_C_Receptacle_USB2.0_16P, J2 SM03B-SRSS-TB_LF__SN_, J3 Micro_SD_Card_Det2, J4 SM03B-SRSS-TB_LF__SN_, J5 USB_C_Receptacle_USB2.0_16P, J6 USB_C_Receptacle_USB2.0_16P, U1 RP2350B, U10 W25Q128JVS, U11 W25Q128JVS, U12 RP2350B, U13 AP2112K-3.3, U14 AP2112K-3.3, U15 W25Q128JVS, U2 STM32H723VGTx, U3 AP2112K-3.3, U4 BMI088, U4 BMP581, U5 BMM350, U6 BMI088, U7 SY8205FCC, U8 AP2112K-3.3, U9 AP2112K-1.8, Y1 ABM8-272-T3, Y2 ABM8-272-T3

Commit message: 27 feb update
Parts:
- added C43: 100nF, Capacitor_SMD:C_0201_0603Metric, F.Cu at (16.4, 111.0)
- added C43: 1uF, Capacitor_SMD:C_1206_3216Metric_Pad1.33x1.80mm_HandSolder, F.Cu at (250.3, 102.3)
- added C44: 100nF, Capacitor_SMD:C_0201_0603Metric, F.Cu at (16.4, 112.8)
- added C44: 10uF, Capacitor_SMD:C_1206_3216Metric_Pad1.33x1.80mm_HandSolder, F.Cu at (196.1, 127.8)
- added C44: 10uF, Capacitor_SMD:C_1206_3216Metric_Pad1.33x1.80mm_HandSolder, F.Cu at (231.1, 92.5)
- added C45: 22uF, Capacitor_SMD:C_1206_3216Metric_Pad1.33x1.80mm_HandSolder, F.Cu at (231.1, 95.8)
- added C45: 22uF, Capacitor_SMD:C_1206_3216Metric_Pad1.33x1.80mm_HandSolder, F.Cu at (196.1, 131.1)
- added C45: 100nF, Capacitor_SMD:C_0201_0603Metric, F.Cu at (16.4, 114.5)
- added C46: 100nF, Capacitor_SMD:C_0201_0603Metric, F.Cu at (18.8, 111.0)
- added C46: 10uF, Capacitor_SMD:C_1206_3216Metric_Pad1.33x1.80mm_HandSolder, F.Cu at (256.7, 82.4)
- added C47: 100nF, Capacitor_SMD:C_0201_0603Metric, F.Cu at (18.8, 112.8)
- added C47: 22uF, Capacitor_SMD:C_1206_3216Metric_Pad1.33x1.80mm_HandSolder, F.Cu at (256.7, 85.8)
- added C48: 10uF, Capacitor_SMD:C_1206_3216Metric_Pad1.33x1.80mm_HandSolder, F.Cu at (271.2, 82.4)
- added C48: 4.7uf, Capacitor_SMD:C_0603_1608Metric, F.Cu at (17.2, 116.6)
- added C49: 22uF, Capacitor_SMD:C_1206_3216Metric_Pad1.33x1.80mm_HandSolder, F.Cu at (271.2, 85.8)
- added C49: 100nF, Capacitor_SMD:C_0201_0603Metric, F.Cu at (18.8, 114.5)
- added C50: 1uF, Capacitor_SMD:C_1206_3216Metric_Pad1.33x1.80mm_HandSolder, F.Cu at (250.3, 105.7)
- added C50: 1uF, Capacitor_SMD:C_0201_0603Metric, F.Cu at (21.3, 111.0)
- added C51: 1uF, Capacitor_SMD:C_1206_3216Metric_Pad1.33x1.80mm_HandSolder, F.Cu at (256.7, 89.1)
- added C51: 2.2uF, Capacitor_SMD:C_0201_0603Metric, F.Cu at (21.3, 112.8)
- added C52: 2.2uF, Capacitor_SMD:C_0201_0603Metric, F.Cu at (21.3, 114.5)
- added C52: 1uF, Capacitor_SMD:C_1206_3216Metric_Pad1.33x1.80mm_HandSolder, F.Cu at (256.7, 92.5)
- added C53: 1uF, Capacitor_SMD:C_1206_3216Metric_Pad1.33x1.80mm_HandSolder, F.Cu at (271.2, 89.1)
- added C54: 1uF, Capacitor_SMD:C_1206_3216Metric_Pad1.33x1.80mm_HandSolder, F.Cu at (271.2, 92.5)
- added C55: 1uF, Capacitor_SMD:C_1206_3216Metric_Pad1.33x1.80mm_HandSolder, F.Cu at (231.1, 99.2)
- added C55: 1uF, Capacitor_SMD:C_1206_3216Metric_Pad1.33x1.80mm_HandSolder, F.Cu at (196.1, 134.4)
- added C56: 1uF, Capacitor_SMD:C_1206_3216Metric_Pad1.33x1.80mm_HandSolder, F.Cu at (231.1, 102.5)
- added C56: 2.2uF, Capacitor_SMD:C_0201_0603Metric, F.Cu at (233.7, 108.5)
- added C57: 0.22uF, Capacitor_SMD:C_0201_0603Metric, F.Cu at (236.7, 111.5)
- added C58: 4.7uF, Capacitor_SMD:C_0201_0603Metric, F.Cu at (230.9, 113.5)
- added C59: 0.22uF, Capacitor_SMD:C_0201_0603Metric, F.Cu at (230.9, 115.2)
- added C60: 4.7uF, Capacitor_SMD:C_0201_0603Metric, F.Cu at (230.9, 117.0)
- added C61: 4.7uF, Capacitor_SMD:C_0201_0603Metric, F.Cu at (230.9, 118.8)
- added C62: 0.22uF, Capacitor_SMD:C_0201_0603Metric, F.Cu at (230.9, 120.5)
- added C63: 10uF, Capacitor_SMD:C_0201_0603Metric, F.Cu at (233.3, 113.5)
- added C64: 0.22uF, Capacitor_SMD:C_0201_0603Metric, F.Cu at (233.3, 115.2)
- added C65: 0.22uF, Capacitor_SMD:C_0201_0603Metric, F.Cu at (233.3, 117.0)
- added C66: 20pF, Capacitor_SMD:C_0201_0603Metric, F.Cu at (233.3, 118.8)
- added C67: 20pF, Capacitor_SMD:C_0201_0603Metric, F.Cu at (233.3, 120.5)
- added C68: 0.22uF, Capacitor_SMD:C_0201_0603Metric, F.Cu at (235.8, 113.5)
- added C69: 2.2uF, Capacitor_SMD:C_0201_0603Metric, F.Cu at (235.8, 115.2)
- added C70: 4.7uF, Capacitor_SMD:C_0201_0603Metric, F.Cu at (235.8, 117.0)
- added C71: 10uF, Capacitor_SMD:C_0201_0603Metric, F.Cu at (235.8, 118.8)
- added C72: 4.7uF, Capacitor_SMD:C_0201_0603Metric, F.Cu at (235.8, 120.5)
- added C73: 0.22uF, Capacitor_SMD:C_0201_0603Metric, F.Cu at (238.2, 113.5)
- added C74: 10uF, Capacitor_SMD:C_0201_0603Metric, F.Cu at (238.2, 115.2)
- added C75: 12pF, Capacitor_SMD:C_0201_0603Metric, F.Cu at (238.2, 117.0)
- added C76: 12pF, Capacitor_SMD:C_0201_0603Metric, F.Cu at (238.2, 118.8)
- added C77: 0.22uF, Capacitor_SMD:C_0201_0603Metric, F.Cu at (238.2, 120.5)
- added C78: 0.22uF, Capacitor_SMD:C_0201_0603Metric, F.Cu at (240.7, 113.5)
- added C79: 10uF, Capacitor_SMD:C_0201_0603Metric, F.Cu at (240.7, 115.2)
- added C80: 0.22uF, Capacitor_SMD:C_0201_0603Metric, F.Cu at (240.7, 117.0)
- added C81: 0.22uF, Capacitor_SMD:C_0201_0603Metric, F.Cu at (240.7, 118.8)
- added C82: ~, Capacitor_SMD:C_0201_0603Metric, F.Cu at (240.7, 120.5)
- added D11: BZV55B5V1, Diode_SMD:D_MiniMELF, F.Cu at (224.9, 82.4)
- added D11: BZV55B5V1, Diode_SMD:D_MiniMELF, F.Cu at (196.3, 114.4)
- added D12: BZV55B5V1, Diode_SMD:D_MiniMELF, F.Cu at (196.3, 117.7)
- added D12: BZV55B5V1, Diode_SMD:D_MiniMELF, F.Cu at (224.9, 85.7)
- added D13: BZV55B5V1, Diode_SMD:D_MiniMELF, F.Cu at (224.9, 89.1)
- added D14: BZV55B5V1, Diode_SMD:D_MiniMELF, F.Cu at (224.9, 92.4)
- added D15: BZV55B5V1, Diode_SMD:D_MiniMELF, F.Cu at (224.9, 95.8)
- added D16: BZV55B5V1, Diode_SMD:D_MiniMELF, F.Cu at (265.1, 89.1)
- added D17: BZV55B5V1, Diode_SMD:D_MiniMELF, F.Cu at (265.1, 92.4)
- added D18: BZV55B5V1, Diode_SMD:D_MiniMELF, F.Cu at (250.5, 89.1)
- added D19: BZV55B5V1, Diode_SMD:D_MiniMELF, F.Cu at (250.5, 92.4)
- added D20: BZV55B5V1, Diode_SMD:D_MiniMELF, F.Cu at (224.9, 99.1)
- added D20: BZV55B5V1, Diode_SMD:D_MiniMELF, F.Cu at (196.3, 121.1)
- added D21: BZV55B5V1, Diode_SMD:D_MiniMELF, F.Cu at (196.3, 124.4)
- added D21: BZV55B5V1, Diode_SMD:D_MiniMELF, F.Cu at (224.9, 102.4)
- added D22: LED, LED_SMD:LED_1206_3216Metric, F.Cu at (209.3, 114.4)
- added D23: LED, LED_SMD:LED_1206_3216Metric_Pad1.42x1.75mm_HandSolder, F.Cu at (235.5, 149.3)
- added D24: BAT54C, Package_TO_SOT_SMD:SOT-23, F.Cu at (202.0, 114.9)
- added D25: BAT54C, Package_TO_SOT_SMD:SOT-23, F.Cu at (202.0, 119.4)
- added D4: BZV55B5V1, Diode_SMD:D_MiniMELF, F.Cu at (265.1, 82.4)
- added D5: BZV55B5V1, Diode_SMD:D_MiniMELF, F.Cu at (265.1, 85.7)
- added D6: BZV55B5V1, Diode_SMD:D_MiniMELF, F.Cu at (250.5, 82.4)
- added D7: BZV55B5V1, Diode_SMD:D_MiniMELF, F.Cu at (250.5, 85.7)
- added F1: 50, 2026-02-20_12-25-28:FUSE_PTS1206_EAT, F.Cu at (169.2, 148.4)
- added FB1: 120, Inductor_SMD:L_0402_1005Metric, F.Cu at (179.2, 147.7)
- added FB2: 120, Inductor_SMD:L_0402_1005Metric, F.Cu at (179.2, 149.7)
- added J6: USB_C_Receptacle_USB2.0_16P, Connector_USB:USB_C_Receptacle_G-Switch_GT-USB-7010ASV, F.Cu at (233.9, 86.1)
- added J7: Conn_Coaxial, Connector_Coaxial:SMA_Amphenol_901-143_Horizontal, F.Cu at (226.5, 73.9)
- added L5: 4.7UH, Inductor_SMD:L_0201_0603Metric_Pad0.64x0.40mm_HandSolder, F.Cu at (188.3, 147.5)
- added PROG1: DNP, Resistor_SMD:R_0402_1005Metric_Pad0.72x0.64mm_HandSolder, F.Cu at (210.5, 117.1)
- added Q1: DMG2302U, Package_TO_SOT_SMD:SOT-23, F.Cu at (202.0, 123.8)
- added R13: 100, Resistor_SMD:R_0201_0603Metric, F.Cu at (185.6, 147.5)
- added R17: 470, Resistor_SMD:R_0201_0603Metric_Pad0.64x0.40mm_HandSolder, F.Cu at (233.9, 151.8)
- added R19: DNP, Resistor_SMD:R_0603_1608Metric, F.Cu at (208.4, 125.4)
- added R21: R, Resistor_SMD:R_01005_0402Metric_Pad0.57x0.30mm_HandSolder, F.Cu at (241.1, 85.2)
- added R22: R, Resistor_SMD:R_01005_0402Metric_Pad0.57x0.30mm_HandSolder, F.Cu at (241.1, 86.8)
- added R25: DNF, Resistor_SMD:R_0603_1608Metric, F.Cu at (17.2, 119.1)
- added R26: 10, Resistor_SMD:R_0201_0603Metric_Pad0.64x0.40mm_HandSolder, F.Cu at (20.6, 116.2)
- added R27: 10, Resistor_SMD:R_0201_0603Metric_Pad0.64x0.40mm_HandSolder, F.Cu at (20.6, 118.0)
- added R28: 64, Resistor_SMD:R_0201_0603Metric, F.Cu at (243.6, 85.2)
- added R28: 64, Resistor_SMD:R_0201_0603Metric, F.Cu at (185.6, 149.3)
- added R29: 64, Resistor_SMD:R_0201_0603Metric, F.Cu at (258.6, 95.0)
- added R30: 64, Resistor_SMD:R_0201_0603Metric, F.Cu at (273.2, 95.0)
- added R32: 470, Resistor_SMD:R_0201_0603Metric, F.Cu at (207.7, 117.0)
- added R33: 100, Resistor_SMD:R_0201_0603Metric, F.Cu at (207.7, 118.7)
- added R4: DNP, Resistor_SMD:R_0603_1608Metric, F.Cu at (208.4, 122.9)
- added U13: TPS2113ADRBR, TPS2113ADRBR:SON65P300X300X100-9N, F.Cu at (250.4, 96.4)
- added U14: TLV75733PDRV, Package_SON:WSON-6-1EP_2x2mm_P0.65mm_EP1x1.6mm, F.Cu at (182.5, 148.5)
- added U14: TLV75733PDRV, Package_SON:WSON-6-1EP_2x2mm_P0.65mm_EP1x1.6mm, F.Cu at (241.6, 82.6)
- added U16: MAX-M10S-00B, MAX-M10S-00B:XCVR_MAX-M10S-00B, F.Cu at (238.8, 67.2)
- added U17: MKL02Z32VFG4, Package_DFN_QFN:QFN-16-1EP_3x3mm_P0.5mm_EP1.9x1.9mm, F.Cu at (237.1, 100.5)
- added U18: W25Q64JVSSIM, 2026-02-19_13-01-05:SOIC_208MIL_WIN, F.Cu at (239.3, 94.3)
- added U19: TLV75733PDRV, Package_SON:WSON-6-1EP_2x2mm_P0.65mm_EP1x1.6mm, F.Cu at (255.5, 96.0)
- added U2: MIMXRT1062DVJ6B, MIMXRT1062DVJ6B:BGA196C80P14X14_1200X1200X152N, F.Cu at (255.4, 68.9)
- added U20: TLV75733PDRV, Package_SON:WSON-6-1EP_2x2mm_P0.65mm_EP1x1.6mm, F.Cu at (270.1, 96.0)
- added U22: TLV75733PDRV, Package_SON:WSON-6-1EP_2x2mm_P0.65mm_EP1x1.6mm, F.Cu at (255.1, 102.5)
- added U3: TPS2113ADRBR, TPS2113ADRBR:SON65P300X300X100-9N, F.Cu at (264.9, 96.4)
- added U8: TPS2113ADRBR, TPS2113ADRBR:SON65P300X300X100-9N, F.Cu at (242.8, 100.1)
- added U8: TPS2113ADRBR, TPS2113ADRBR:SON65P300X300X100-9N, F.Cu at (175.3, 148.9)
- added Y3: ABMM2-32.768MHZ-E2F-T, ABMM2-32.768MHZ-E2F-T:XTAL_ABMM2-32.768MHZ-E2F-T, F.Cu at (196.5, 140.0)
- added Y4: 24MHZ, Crystal:Crystal_SMD_Abracon_ABM3-2Pin_5.0x3.2mm, F.Cu at (196.9, 146.5)
Connections:
- J3 pad 10: unconnected-(J3-DET_A-Pad10) -> TEL-DET
- J3 pad 11: unconnected-(J3-SHIELD-Pad11) -> GND
- J3 pad 2: unconnected-(J3-DAT3/CD-Pad2) -> TEL-CS
- J3 pad 3: unconnected-(J3-CMD-Pad3) -> TEL-MOSI
- J3 pad 4: unconnected-(J3-VDD-Pad4) -> Tel-3.3V
- J3 pad 5: unconnected-(J3-CLK-Pad5) -> TEL-SCK
- J3 pad 6: unconnected-(J3-VSS-Pad6) -> GND
- J3 pad 7: unconnected-(J3-DAT0-Pad7) -> TEL-MISO
- J3 pad 9: unconnected-(J3-DET_B-Pad9) -> TEL-DET
- R14 pad 1: Net-(R13-Pad2) -> unconnected-(R14-Pad1)
- R18 pad 1: Net-(R17-Pad2) -> unconnected-(R18-Pad1)
- U1 pad 81: unconnected-(U1-GND-Pad81) -> GND
- U12 pad 14: unconnected-(U12-GPIO15-Pad14) -> TEL-DET
- U12 pad 16: unconnected-(U12-GPIO16-Pad16) -> TEL-MISO
- U12 pad 17: unconnected-(U12-GPIO17-Pad17) -> TEL-CS
- U12 pad 18: unconnected-(U12-GPIO18-Pad18) -> TEL-SCK
- U12 pad 19: unconnected-(U12-GPIO19-Pad19) -> TEL-MOSI
- U12 pad 81: unconnected-(U12-GND-Pad81) -> GND
- U2 pad 10: Net-(U2-VSS-Pad10) -> GND
- U2 pad 100: unconnected-(U2-VDD-Pad100) -> Net-(C43-Pad1)
- U2 pad 11: unconnected-(U2-VDD-Pad11) -> Net-(C43-Pad1)
- U2 pad 14: unconnected-(U2-NRST-Pad14) -> MPU-NRST
- U2 pad 19: unconnected-(U2-VSSA-Pad19) -> GND
- U2 pad 20: unconnected-(U2-VREF+-Pad20) -> MPU-3.3V
- U2 pad 21: unconnected-(U2-VDDA-Pad21) -> MPU-3.3V
- U2 pad 26: Net-(U2-VSS-Pad10) -> GND
- U2 pad 27: unconnected-(U2-VDD-Pad27) -> Net-(C43-Pad1)
- U2 pad 48: unconnected-(U2-VCAP-Pad48) -> Net-(C52-Pad1)
- U2 pad 49: Net-(U2-VSS-Pad10) -> GND
- U2 pad 50: unconnected-(U2-VDD-Pad50) -> Net-(C43-Pad1)
- U2 pad 73: unconnected-(U2-VCAP-Pad73) -> Net-(C51-Pad1)
- U2 pad 74: Net-(U2-VSS-Pad10) -> GND
- U2 pad 75: unconnected-(U2-VDD-Pad75) -> Net-(C43-Pad1)
- U2 pad 94: unconnected-(U2-BOOT0-Pad94) -> MPU-BOOT0
- U2 pad 99: Net-(U2-VSS-Pad10) -> GND
- U4 pad 8: unconnected-(U4-VSS_2-Pad8) -> GND
- U4 pad 9: unconnected-(U4-VSS_3-Pad9) -> GND
- U5 pad B1: unconnected-(U5-GND-PadB1) -> GND
- U6 pad 6: unconnected-(U6-GNDIO-Pad6) -> GND
Other:
- copper layers 2 -> 4

Commit message: 12-March update
Parts:
- removed the C41 at (120.1, 137.0)
- removed C42: 100nf, Capacitor_SMD:C_0402_1005Metric
- removed the C43 at (16.4, 111.0)
- removed the C44 at (16.4, 112.8)
- removed the C45 at (16.4, 114.5)
- removed the C46 at (18.8, 111.0)
- removed the C47 at (18.8, 112.8)
- removed the C48 at (17.2, 116.6)
- removed the C49 at (18.8, 114.5)
- removed the C50 at (21.3, 111.0)
- removed the C52 at (21.3, 114.5)
- removed the J6 at (233.9, 86.1)
- removed the J6 at (128.9, 113.4)
- removed PROG1: DNP, Resistor_SMD:R_0402_1005Metric_Pad0.72x0.64mm_HandSolder
- removed the R17 at (145.9, 88.8)
- removed the R19 at (177.1, 69.6)
- removed the R25 at (17.2, 119.1)
- removed the R26 at (20.6, 116.2)
- removed the R27 at (20.6, 118.0)
- removed the R4 at (26.5, 46.4)
- removed R5: 33, Resistor_SMD:R_0201_0603Metric_Pad0.64x0.40mm_HandSolder
- removed U15: W25Q128JVS, Package_SO:SOIC-8_5.3x5.3mm_P1.27mm
- removed the U2 at (78.2, 50.6)
- removed the U4 at (79.2, 64.6)
- added BZ1: Buzzer, MLT-8530_JHE:MLT-8530_JHE_1, F.Cu at (72.6, 131.1)
- added C16: 100nF, Capacitor_SMD:C_01005_0402Metric, F.Cu at (197.4, 67.6)
- added C38: ~, Connector_PinSocket_1.00mm:1x10pin, F.Cu at (24.1, 158.4)
- added C41: 0.22uF, Capacitor_SMD:C_0201_0603Metric, F.Cu at (201.8, 74.1)
- added C41: 1uF, Capacitor_SMD:C_0402_1005Metric, F.Cu at (128.9, 167.5)
- added C52: 47UF, Capacitor_SMD:C_0402_1005Metric, F.Cu at (144.8, 136.6)
- added C52: 100nF, Capacitor_SMD:C_01005_0402Metric, F.Cu at (131.4, 168.9)
- added C53: 10pF, Capacitor_SMD:C_0201_0603Metric, F.Cu at (114.3, 168.1)
- added C83: 2.2uF, Capacitor_SMD:C_0201_0603Metric, F.Cu at (180.7, 112.5)
- added C84: 100NF, Capacitor_SMD:C_0201_0603Metric, F.Cu at (203.5, 55.2)
- added C85: 100NF, Capacitor_SMD:C_0201_0603Metric, F.Cu at (203.5, 56.9)
- added C86: 100NF, Capacitor_SMD:C_0201_0603Metric, F.Cu at (203.5, 58.7)
- added C87: 100NF, Capacitor_SMD:C_0201_0603Metric, F.Cu at (203.5, 60.4)
- added C88: 100NF, Capacitor_SMD:C_0201_0603Metric, F.Cu at (205.9, 55.2)
- added C89: 100NF, Capacitor_SMD:C_0201_0603Metric, F.Cu at (205.9, 56.9)
- added D1: 1N4148WT, Diode_SMD:D_SOD-523, F.Cu at (45.3, 36.0)
- added D2: WS2812, LED_SMD:LED_WS2812_PLCC6_5.0x5.0mm_P1.6mm, F.Cu at (89.9, 55.2)
- added D2: WS2812B-2020, LED_SMD:LED_WS2812B-2020_PLCC4_2.0x2.0mm, F.Cu at (61.6, 132.8)
- added D26: 1N914WT, Diode_SMD:D_SOD-523, B.Cu at (92.1, 60.3)
- added D27: 1N914WT, Diode_SMD:D_SOD-523, B.Cu at (92.1, 62.9)
- added D28: 1N914WT, Diode_SMD:D_SOD-523, B.Cu at (135.3, 60.3)
- added D29: 1N914WT, Diode_SMD:D_SOD-523, B.Cu at (135.3, 62.9)
- added D30: 1N4148WT, Diode_SMD:D_SOD-523, F.Cu at (45.3, 38.5)
- added D31: WS2812, LED_SMD:LED_WS2812_PLCC6_5.0x5.0mm_P1.6mm, F.Cu at (131.6, 55.2)
- added D31: WS2812B-2020, LED_SMD:LED_WS2812B-2020_PLCC4_2.0x2.0mm, F.Cu at (82.7, 132.8)
- added D32: WS2812B-2020, LED_SMD:LED_WS2812B-2020_PLCC4_2.0x2.0mm, F.Cu at (38.9, 132.8)
- added D32: WS2812, LED_SMD:LED_WS2812_PLCC6_5.0x5.0mm_P1.6mm, F.Cu at (110.5, 55.2)
- added G1: SIT1602AI-32-33E-30.000000, SIT1602AI-32-33E-30.000000:OSC_SIT1602AI-32-33E-30.000000, B.Cu at (53.3, 126.4)
- added H1: Batsolderpad, TestPoint:TestPoint_Pad_4.0x4.0mm, F.Cu at (80.0, 144.1)
- added H2: Batsolderpad, TestPoint:TestPoint_Pad_4.0x4.0mm, F.Cu at (87.0, 144.1)
- added IC1: SI4464-B1B-FM, SI4464-B1B-FM:QFN50P400X400X90-21N, F.Cu at (77.3, 110.0)
- added IC3: AT7456E-1, AT7456E:SOP65P640X120-29N, F.Cu at (147.8, 130.0)
- added J10: Conn_Coaxial, Connector_Coaxial:SMA_Amphenol_901-143_Horizontal, F.Cu at (99.1, 109.2)
- added J11: Conn_Coaxial, Connector_Coaxial:SMA_Amphenol_901-143_Horizontal, F.Cu at (110.5, 22.9)
- added J6: USB_C_Receptacle_USB2.0_16P, Connector_USB:USB_C_Receptacle_G-Switch_GT-USB-7010ASV, F.Cu at (50.7, 110.5)
- added J8: S8411-45R, S8411-45R:HARWIN_S8411-45R, B.Cu at (77.6, 132.1)
- added J9: Conn_01x02, Connector_PinSocket_1.00mm:PinSocket_1x02_P1.00mm_Vertical, F.Cu at (131.5, 173.5)
- added L1: AOTA-B201610S3R3-101-T, AOTA-B201610S3R3-101-T:AOTAB201610S3R3101T, F.Cu at (124.4, 174.1)
- added L2: SPM4012T-2R2M, SPM4012T-2R2M:IND_SPM4012T-2R2M, F.Cu at (124.6, 152.8)
- added NAV-QSPI_SS: R, Resistor_SMD:R_2010_5025Metric_Pad1.40x2.65mm_HandSolder, F.Cu at (85.1, 61.6)
- added NAV-RESET: R, Resistor_SMD:R_2010_5025Metric_Pad1.40x2.65mm_HandSolder, F.Cu at (94.0, 61.6)
- added OSD-VIN1: Solderpad, TestPoint:TestPoint_Pad_1.5x1.5mm, F.Cu at (154.1, 133.8)
- added OSD-VOUT1: Solderpad, TestPoint:TestPoint_Pad_1.5x1.5mm, F.Cu at (154.1, 137.4)
- added Q2: 2N7002, Package_TO_SOT_SMD:SOT-23, F.Cu at (212.0, 56.5)
- added Q3: 2N7002, Package_TO_SOT_SMD:SOT-23, B.Cu at (93.0, 65.7)
- added Q4: 2N7002, Package_TO_SOT_SMD:SOT-23, B.Cu at (134.6, 66.0)
- added R18: DNP, Resistor_SMD:R_0603_1608Metric, F.Cu at (196.5, 75.0)
- added R21: 5.1k, Resistor_SMD:R_0201_0603Metric, F.Cu at (180.7, 116.2)
- added R22: 5.1k, Resistor_SMD:R_0201_0603Metric, F.Cu at (180.7, 118.0)
- added R25: 4.7K, Resistor_SMD:R_0201_0603Metric, F.Cu at (205.9, 58.7)
- added R25: 4.7K, Resistor_SMD:R_0201_0603Metric, F.Cu at (125.4, 177.3)
- added R26: 4.7K, Resistor_SMD:R_0201_0603Metric, F.Cu at (131.5, 165.4)
- added R26: 4.7K, Resistor_SMD:R_0201_0603Metric, F.Cu at (205.9, 60.4)
- added R27: 4.7K, Resistor_SMD:R_0201_0603Metric, F.Cu at (125.4, 179.1)
- added R27: 4.7K, Resistor_SMD:R_0201_0603Metric, F.Cu at (208.4, 55.2)
- added R31: 4.7K, Resistor_SMD:R_0201_0603Metric, F.Cu at (131.5, 167.2)
- added R31: 4.7K, Resistor_SMD:R_0201_0603Metric, F.Cu at (208.4, 56.9)
- added R34: 10, Resistor_SMD:R_0201_0603Metric_Pad0.64x0.40mm_HandSolder, F.Cu at (139.9, 64.1)
- added R35: 10k\, Resistor_SMD:R_0201_0603Metric, F.Cu at (67.7, 182.9)
- added R36: 4.7K, Resistor_SMD:R_0201_0603Metric, F.Cu at (208.4, 58.7)
- added R37: 4.7K, Resistor_SMD:R_0201_0603Metric, F.Cu at (208.4, 60.4)
- added TEL-QSPI_SS: R, Resistor_SMD:R_2010_5025Metric_Pad1.40x2.65mm_HandSolder, F.Cu at (127.1, 61.6)
- added TEL-RESET: R, Resistor_SMD:R_2010_5025Metric_Pad1.40x2.65mm_HandSolder, F.Cu at (136.7, 61.6)
- added TR1: ADT1-1WT, RF_Mini-Circuits:Mini-Circuits_CD542_H2.84mm, B.Cu at (88.3, 109.2)
- added U21: DS3231M, Package_SO:SOIC-16W_7.5x10.3mm_P1.27mm, B.Cu at (56.2, 135.9)
- added Y5: ABMM2-105-27.000MHZ-T, ABMM2-105-27.000MHZ-T:XTAL_ABMM2-105-27.000MHZ-T, F.Cu at (155.6, 128.2)
- C37: value 100nf -> 1uF; footprint Capacitor_SMD:C_1206_3216Metric_Pad1.33x1.80mm_HandSolder -> Capacitor_SMD:C_0402_1005Metric
- C39: value 1uf -> 1uF; footprint Capacitor_SMD:C_1206_3216Metric_Pad1.33x1.80mm_HandSolder -> Capacitor_SMD:C_0402_1005Metric
- C40: value 10uf -> 1uF
- C51: value 2.2uF -> 50nF
- C52: footprint Capacitor_SMD:C_1206_3216Metric_Pad1.33x1.80mm_HandSolder -> Capacitor_SMD:C_0201_0603Metric
- L3: value 3.3uH-XAL7030-332ME -> AOTA-B201610S3R3-101-T; footprint Inductor_SMD:L_6.3x6.3_H3 -> AOTA-B201610S3R3-101-T:AOTAB201610S3R3101T
- R23: value 110k -> 44.2k; footprint Resistor_SMD:R_0508_1220Metric_Pad1.12x2.15mm_HandSolder -> Resistor_SMD:R_0402_1005Metric
- R24: value 15k -> 6.04k; footprint Resistor_SMD:R_0508_1220Metric -> Resistor_SMD:R_0402_1005Metric
- U1: value RP2350B -> Navigation
- U10, U11, U16, U17, U18, Y3: moved to B.Cu
- U12: value RP2350B -> Telemetry
- U2: value MIMXRT1062DVJ6B -> MPU
- moved U16 209.8 mm to (40.6, 135.9), turned to 180 degrees
- moved U8 205.1 mm to (45.6, 156.6)
- moved U17 198.6 mm to (39.1, 116.3), turned to 180 degrees
- moved U14 192.2 mm to (64.4, 156.9)
- moved U18 154.0 mm to (90.3, 55.2), turned to 180 degrees
- moved U2 148.0 mm to (110.5, 38.9), turned to 45 degrees
- moved J7 145.5 mm to (97.8, 141.6), turned to -90 degrees
- moved D13 140.9 mm to (112.7, 174.2)
- moved D14 140.9 mm to (112.7, 177.6)
- moved D15 140.9 mm to (112.7, 180.9)
- moved Y4 135.5 mm to (120.0, 34.9), turned to -45 degrees
- moved Y3 123.5 mm to (117.5, 45.1), turned to 135 degrees
- moved C51 114.7 mm to (131.5, 144.4)
- moved C14 106.6 mm to (70.1, 191.1)
- moved C15 106.6 mm to (70.1, 192.7)
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Connections:
- C37 pad 1: Net-(U7-BS) -> Nav-3.3V
- C37 pad 2: Net-(U7-LX) -> GND
- C39 pad 1: Net-(U7-VCC) -> Tel-3.3V
- C40 pad 1: VCC -> Tel-5V-stable
- C51 pad 1: Net-(C51-Pad1) -> GND
- C51 pad 2: GND -> Net-(U7-SS)
- J1 pad A6: Net-(D2-A) -> Net-(D1-A)
- J1 pad A7: Net-(D1-A) -> Net-(D30-A)
- J1 pad B6: Net-(D2-A) -> Net-(D1-A)
- J1 pad B7: Net-(D1-A) -> Net-(D30-A)
- J7 pad 1: Net-(J7-In) -> Net-(IC1-TX)
- J7 pad 2: Net-(J7-Ext) -> GND
- L3 pad 1: +5V -> Net-(U1-VREG_LX)
- L3 pad 2: Net-(U7-LX) -> Nav-3.3V
- R14 pad 1: unconnected-(R14-Pad1) -> Net-(DNP3-Pad2)
- R19 pad 1: Nav-RUN -> Net-(D26-K)
- R20 pad 1: Net-(R19-Pad2) -> Net-(DNP2-Pad2)
- R23 pad 1: +5V -> Net-(U7-FB)
- R23 pad 2: Net-(U7-FB) -> +5V
- R24 pad 1: GND -> Net-(U7-FB)
- R24 pad 2: Net-(U7-FB) -> GND
- U1 pad 1: unconnected-(U1-GPIO4-Pad1) -> NAV-SDA
- U1 pad 11: unconnected-(U1-GPIO12-Pad11) -> NAV-MPU-MISO
- U1 pad 12: unconnected-(U1-GPIO13-Pad12) -> NAV-MPU-CS
- U1 pad 13: unconnected-(U1-GPIO14-Pad13) -> NAV-TEL-SDA
- U1 pad 14: unconnected-(U1-GPIO15-Pad14) -> NAV-TEL-SCL
- U1 pad 16: unconnected-(U1-GPIO16-Pad16) -> NAV-MISO
- U1 pad 18: unconnected-(U1-GPIO18-Pad18) -> NAV-SCK
- U1 pad 19: unconnected-(U1-GPIO19-Pad19) -> NAV-MOSI
- U1 pad 2: unconnected-(U1-GPIO5-Pad2) -> NAV-SCL
- U1 pad 20: unconnected-(U1-GPIO20-Pad20) -> BMI088-INT-3
- U1 pad 21: unconnected-(U1-GPIO21-Pad21) -> BMI088-INT-4
- U1 pad 22: unconnected-(U1-GPIO22-Pad22) -> BMM350-INT
- U1 pad 23: unconnected-(U1-GPIO23-Pad23) -> BMP581-INT
- U1 pad 3: unconnected-(U1-GPIO6-Pad3) -> Nav-stat
- U1 pad 42: unconnected-(U1-GPIO33-Pad42) -> NAV-GYRO-CS
- U1 pad 46: unconnected-(U1-GPIO37-Pad46) -> NAV-ACC-CS
- U1 pad 52: unconnected-(U1-GPIO41/ADC1-Pad52) -> NAV-RADIO-CS
- U1 pad 6: unconnected-(U1-GPIO8-Pad6) -> BMI088-INT-1
- U1 pad 7: unconnected-(U1-GPIO9-Pad7) -> BMI088-INT-2
- U1 pad 78: unconnected-(U1-GPIO1-Pad78) -> GPS-RESET
- U1 pad 79: unconnected-(U1-GPIO2-Pad79) -> Timepulse
- U1 pad 8: unconnected-(U1-GPIO10-Pad8) -> NAV-MPU-SCK
- U1 pad 80: unconnected-(U1-GPIO3-Pad80) -> RTC-1MHZ
- U1 pad 9: unconnected-(U1-GPIO11-Pad9) -> NAV-MPU-MOSI
- U10 pad 1: Nav-QSPI_SS -> Tel-QSPI_SS
- U10 pad 2: Nav-QSPI_SD1 -> Tel-QSPI_SD1
- U10 pad 3: Nav-QSPI_SD2 -> Tel-QSPI_SD2
- U10 pad 5: Nav-QSPI_SD0 -> Tel-QSPI_SD0
- U10 pad 6: Nav-QSPI_SCLK -> Tel-QSPI_SCLK
- U10 pad 7: Nav-QSPI_SD3 -> Tel-QSPI_SD3
- U10 pad 8: Nav-3.3V -> Tel-3.3V
- U11 pad 1: Nav-GPIO0 -> Nav-QSPI_SS
- U12 pad 11: unconnected-(U12-GPIO12-Pad11) -> TEL-MPU-MISO
- U12 pad 12: unconnected-(U12-GPIO13-Pad12) -> TEL-MPU-CS
- U12 pad 13: unconnected-(U12-GPIO14-Pad13) -> NAV-TEL-SDA
- U12 pad 14: TEL-DET -> NAV-TEL-SCL
- U12 pad 2: unconnected-(U12-GPIO5-Pad2) -> TEL-RADIO-SC
- U12 pad 20: unconnected-(U12-GPIO20-Pad20) -> TEL-INT
- U12 pad 21: unconnected-(U12-GPIO21-Pad21) -> TEL-SDN
- U12 pad 22: unconnected-(U12-GPIO22-Pad22) -> TEL-DET
- U12 pad 77: unconnected-(U12-GPIO0-Pad77) -> RTC-1MHZ
- U12 pad 78: unconnected-(U12-GPIO1-Pad78) -> Tel-stat
- U12 pad 8: unconnected-(U12-GPIO10-Pad8) -> TEL-MPU-SCK
- U12 pad 9: unconnected-(U12-GPIO11-Pad9) -> TEL-MPU-MOSI
- U13 pad 7: Net-(U13-OUT) -> Tel-5V-stable
- U16 pad 11: Net-(J7-In) -> Net-(J11-In)
- U16 pad 14: Net-(J7-Ext) -> unconnected-(U16-VCC_RF-Pad14)
- U16 pad 16: unconnected-(U16-SDA-Pad16) -> Nav-SDA
- U16 pad 17: unconnected-(U16-SCL-Pad17) -> Nav-SCL
- U16 pad 4: unconnected-(U16-TIMEPULSE-Pad4) -> Timepulse
- U16 pad 6: unconnected-(U16-V_BCKP-Pad6) -> Nav-3.3V
- U16 pad 7: unconnected-(U16-V_IO-Pad7) -> Nav-3.3V
- U16 pad 8: GND -> Nav-3.3V
- U16 pad 9: unconnected-(U16-~{RESET}-Pad9) -> Net-(Q2-D)
- U19 pad 4: Net-(U13-OUT) -> Tel-5V-stable
- U19 pad 6: Net-(U13-OUT) -> Tel-5V-stable
- U2 pad D3: unconnected-(U2B-GPIO_EMC_24-PadD3) -> Net-(BZ1-+)
- U2 pad G11: unconnected-(U2A-GPIO_AD_B0_03-PadG11) -> MPU-CS
- U2 pad G2: unconnected-(U2B-GPIO_EMC_23-PadG2) -> MPU-stat
- U2 pad H10: unconnected-(U2A-GPIO_AD_B0_01-PadH10) -> MPI-MOSI
- U2 pad J1: unconnected-(U2A-GPIO_SD_B0_02-PadJ1) -> TEL-MPU-MOSI
- U2 pad J3: unconnected-(U2A-GPIO_SD_B0_01-PadJ3) -> TEL-MPU-CS
- U2 pad J4: unconnected-(U2A-GPIO_SD_B0_00-PadJ4) -> TEL-MPU-SCK
- U2 pad K1: unconnected-(U2A-GPIO_SD_B0_03-PadK1) -> TEL-MPU-MISO
- U2 pad K14: unconnected-(U2A-GPIO_AD_B0_12-PadK14) -> OSD-RESET
- U2 pad L3: unconnected-(U2A-GPIO_SD_B1_06-PadL3) -> NAV-MPU-CS
- U2 pad L4: unconnected-(U2A-GPIO_SD_B1_07-PadL4) -> NAV-MPU-SCK
- U2 pad M11: unconnected-(U2A-GPIO_AD_B0_02-PadM11) -> MPU-MISO
- U2 pad M14: unconnected-(U2A-GPIO_AD_B0_00-PadM14) -> MPU-SCK
- U2 pad N4: unconnected-(U2A-GPIO_SD_B1_09-PadN4) -> NAV-MPU-MISO
- U2 pad N7: unconnected-(U2B-USB_OTG2_DN-PadN7) -> Net-(J9-Pin_2)
- U2 pad P3: unconnected-(U2A-GPIO_SD_B1_08-PadP3) -> NAV-MPU-MOSI
- U2 pad P7: unconnected-(U2B-USB_OTG2_DP-PadP7) -> Net-(J9-Pin_1)
- U20 pad 4: Net-(U20-EN) -> Nav-5V-stable
- U20 pad 6: Net-(U20-EN) -> Nav-5V-stable
- U3 pad 7: Net-(U20-EN) -> Nav-5V-stable
- U4 pad 1: unconnected-(U4-VDDIO-Pad1) -> Nav-3.3V
- U4 pad 10: unconnected-(U4-VDD-Pad10) -> Nav-3.3V
- U4 pad 2: unconnected-(U4-SCK-Pad2) -> Nav-SCL
- U4 pad 3: unconnected-(U4-VSS_1-Pad3) -> GND
- U4 pad 4: unconnected-(U4-SDI-Pad4) -> Nav-SDA
- U4 pad 5: unconnected-(U4-SDO-Pad5) -> Nav-3.3V
- U4 pad 6: unconnected-(U4-CSB-Pad6) -> Nav-3.3V
- U4 pad 7: unconnected-(U4-INT-Pad7) -> BMP581-INT
- U5 pad A1: unconnected-(U5-INT-PadA1) -> BMM350-INT
- U5 pad A2: unconnected-(U5-SDA-PadA2) -> Nav-SDA
- U5 pad A3: unconnected-(U5-SCK-PadA3) -> Nav-SCL
- U5 pad B2: unconnected-(U5-ADSEL-PadB2) -> GND
- U5 pad B3: unconnected-(U5-VDDIO-PadB3) -> Nav-3.3V
- U5 pad C1: unconnected-(U5-VDD-PadC1) -> Nav-3.3V
- U5 pad C2: unconnected-(U5-CRST-PadC2) -> Net-(U5-CRST)
- U5 pad C3: unconnected-(U5-BYPASS-PadC3) -> GND
- U6 pad 1: unconnected-(U6-INT2-Pad1) -> BMI088-INT-2
- U6 pad 10: unconnected-(U6-SDO2-Pad10) -> NAV-MISO
- U6 pad 11: unconnected-(U6-VDDIO-Pad11) -> Nav-3.3V
- U6 pad 12: unconnected-(U6-INT3-Pad12) -> BMI088-INT-3
- U6 pad 13: unconnected-(U6-INT4-Pad13) -> BMI088-INT-4
- U6 pad 14: unconnected-(U6-~{CSB1}-Pad14) -> NAV-ACC-CS
- U6 pad 15: unconnected-(U6-SDO1-Pad15) -> NAV-MISO
- U6 pad 16: unconnected-(U6-INT1-Pad16) -> BMI088-INT-1
- U6 pad 3: unconnected-(U6-VDD-Pad3) -> Nav-3.3V
- U6 pad 5: unconnected-(U6-~{CSB2}-Pad5) -> NAV-GYRO-CS
- U6 pad 7: unconnected-(U6-PS-Pad7) -> GND
- U6 pad 8: unconnected-(U6-SCK/SCL-Pad8) -> NAV-SCK
- U6 pad 9: unconnected-(U6-SDI/SDA-Pad9) -> NAV-MOSI
- U7 pad 3: VCC -> +24V
- U7 pad 6: Net-(U7-VCC) -> unconnected-(U7-VCC-Pad6)
- U7 pad 7: VCC -> +24V
- U7 pad 8: VCC -> +24V
Other:
- board outline added: 75.6 x 41.9 mm

Commit message: test gpg
Parts:
- removed the C16 at (70.1, 194.4)
- removed C38: 100nF, Capacitor_SMD:C_01005_0402Metric
- removed C38: ~, Connector_PinSocket_1.00mm:1x10pin
- removed the C41 at (201.8, 74.1)
- removed the C44 at (231.1, 92.5)
- removed the C45 at (231.1, 95.8)
- removed C51, C54: 1uF, Capacitor_SMD:C_1206_3216Metric_Pad1.33x1.80mm_HandSolder
- removed C51: 50nF, Capacitor_SMD:C_0201_0603Metric
- removed the C52 at (131.4, 168.9)
- removed the C52 at (256.7, 92.5)
- removed the C53 at (271.2, 89.1)
- removed the C55 at (231.1, 99.2)
- removed the C56 at (231.1, 102.5)
- removed D1, D30: 1N4148WT, Diode_SMD:D_SOD-523
- removed D1, D10, D14 (x2), D15 (x2), D9: BZV55B5V1, Diode_SMD:D_MiniMELF
- removed the D11 at (224.9, 82.4)
- removed the D11 at (119.9, 109.7)
- removed the D12 at (119.9, 113.0)
- removed the D12 at (224.9, 85.7)
- removed the D13 at (119.9, 116.4)
- removed the D2 at (61.6, 132.8)
- removed the D2 at (105.5, 85.5)
- removed the D20 at (224.9, 99.1)
- removed the D21 at (224.9, 102.4)
- removed the D31 at (82.7, 132.8)
- removed the D32 at (38.9, 132.8)
- removed the D4 at (38.4, 159.1)
- removed the D5 at (38.4, 162.4)
- removed the D6 at (147.1, 70.0)
- removed the D7 at (147.1, 73.4)
- removed the L1 at (72.8, 189.5)
- removed L2: SPM4012T-2R2M, SPM4012T-2R2M:IND_SPM4012T-2R2M
- removed L2: 3.3u, Inductor_SMD:L_0201_0603Metric
- removed the R13 at (145.9, 86.3)
- removed R18: 10, Resistor_SMD:R_0201_0603Metric_Pad0.64x0.40mm_HandSolder
- removed R18, R19, R4: DNP, Resistor_SMD:R_0603_1608Metric
- removed the R21 at (129.5, 118.9)
- removed the R21 at (241.1, 85.2)
- removed the R22 at (241.1, 86.8)
- removed the R22 at (129.5, 120.6)
- removed R23: 44.2k, Resistor_SMD:R_0402_1005Metric
- removed R24: 6.04k, Resistor_SMD:R_0402_1005Metric
- removed the R25 at (205.9, 58.7)
- removed the R26 at (205.9, 60.4)
- removed the R27 at (208.4, 55.2)
- removed the R28 at (243.6, 85.2)
- removed the R31 at (208.4, 56.9)
- removed the U13 at (161.9, 95.9)
- removed the U14 at (125.6, 120.5)
- removed the U14 at (64.4, 156.9)
- removed the U3 at (37.8, 166.5)
- removed U7: SY8205FCC, SY8205FCC:VREG_SY8205FCC
- removed the U8 at (60.5, 170.3)
- removed the U8 at (45.6, 156.6)
- added PROG1: DNP, Resistor_SMD:R_2010_5025Metric_Pad1.40x2.65mm_HandSolder, F.Cu at (110.5, 61.6)
- added R5: 33, Resistor_SMD:R_0201_0603Metric_Pad0.64x0.40mm_HandSolder, F.Cu at (91.6, 158.8)
- added U15: TPS54302, Package_TO_SOT_SMD:SOT-23-6, F.Cu at (110.6, 68.9)
- IC1, IC3, J2, J4, U13, U14, U19, U20, U22, U3, U8, Y5: moved to B.Cu
- J8: moved to F.Cu
- U1: value Navigation -> RP2350B
- U12: value Telemetry -> RP2350B
- U2: value MPU -> MIMXRT1062DVJ6B
- moved U20 184.8 mm to (95.4, 35.7), turned to -135 degrees
- moved U3 183.5 mm to (92.7, 33.0), turned to -135 degrees
- moved U22 148.4 mm to (110.5, 69.2), turned to 180 degrees
- moved J2 146.6 mm to (84.8, 48.5), turned to 90 degrees
- moved U14 140.7 mm to (100.0, 34.6), turned to -45 degrees
- moved U16 138.2 mm to (122.9, 24.8)
- moved U8 135.0 mm to (102.7, 32.2), turned to 135 degrees
- moved U19 131.9 mm to (138.1, 35.9), turned to -135 degrees
- moved U13 131.1 mm to (135.2, 33.6), turned to -135 degrees
- moved D3 102.7 mm to (51.4, 152.4)
- moved U17 95.4 mm to (102.5, 45.0), turned to 45 degrees
- moved J3 91.4 mm to (134.8, 89.3), turned to -90 degrees
- moved TR1 79.4 mm to (22.9, 154.3)
- moved J5 68.0 mm to (137.4, 75.4)
- moved U6 61.2 mm to (110.5, 75.6)
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- renumbered NAV-QSPI_SS to DNP1, NAV-RESET to DNP2, TEL-QSPI_SS to DNP3, TEL-RESET to DNP4
Connections:
- J1 pad A6: Net-(D1-A) -> Nav-D+
- J1 pad A7: Net-(D30-A) -> Nav-D-
- J1 pad B6: Net-(D1-A) -> Nav-D+
- J1 pad B7: Net-(D30-A) -> Nav-D-
- J5 pad A6: Net-(D10-A) -> Tel-D+
- J5 pad A7: Net-(D9-A) -> Tel-D-
- J5 pad B6: Net-(D10-A) -> Tel-D+
- J5 pad B7: Net-(D9-A) -> Tel-D-
- J6 pad A6: Net-(D15-A) -> MPU-D+
- J6 pad A7: Net-(D14-A) -> MPU-D-
- J6 pad B6: Net-(D15-A) -> MPU-D+
- J6 pad B7: Net-(D14-A) -> MPU-D-
Other:
- board size 75.6 x 41.9 mm -> 108 x 134 mm
