File: Hardware/MPUBootloader.kicad_sch (KiCad schematic)
At the start: 11 parts, among them J6 USB_C_Receptacle_USB2.0_16P, U14 AP2112K-3.3, U17 MKL02Z32VFG4, U18 W25Q64JVSSIM

Commit message: 27 feb update
Parts:
- removed D11, D12: BZV55B5V1, Diode_SMD:D_MiniMELF, symbol Diode:BZV55B5V1
- removed U14: AP2112K-3.3, Package_TO_SOT_SMD:SOT-23-5, symbol Regulator_Linear:AP2112K-3.3
- added D22: LED, LED_SMD:LED_1206_3216Metric, symbol Device:LED
- added PROG1: DNP, Resistor_SMD:R_0402_1005Metric_Pad0.72x0.64mm_HandSolder, symbol Device:R
- added R32: 470, Resistor_SMD:R_0201_0603Metric, symbol Device:R
- added R33: 100, Resistor_SMD:R_0201_0603Metric, symbol Device:R
- R21, R22: value R -> 5.1k; footprint Resistor_SMD:R_01005_0402Metric_Pad0.57x0.30mm_HandSolder -> Resistor_SMD:R_0201_0603Metric
Connections:
- net GND: now also U17.17 (EPAD), U17.2 (VSS/VREFL), U18.4 (GND), PROG1.2, R33.1
- net MPU-3.3V: now also U18.8 (VCC), D22.2 (A)
- net at J6.B5 (CC2): now also R21.1; no longer R22.1
- net at J6.A5 (CC1): now also R22.1; no longer R21.1
- net 5V-MPU: now reaches U17.1 (VDD/VREFH)
- net at U17.10 (PTB2/IRQ_7): now also PROG1.1
- net PTB3: now reaches U17.11 (PTB3/IRQ_10)
- net PTB3: now also R32.2
- net PTB4: now reaches U17.12 (PTB4/IRQ_11)
- net PTB5: now reaches U17.13 (PTB5/IRQ_12)
- net DNC0: now reaches U17.14 (PTA0/IRQ_0)
- net PTA1: now reaches U17.15 (PTA1/IRQ_1/LPTMR0_ALT1)
- net DNC1: now reaches U17.16 (PTA2)
- net AD_B0_11: now reaches U17.3 (PTA3)
- net AD_B0_11: now also R33.2
- net PTA4: now reaches U17.4 (PTA4)
- net PTA5: now reaches U17.5 (PTA5)
- net PTA6: now reaches U17.6 (PTA6)
- net PTA7: now reaches U17.7 (PTA7/IRQ_4)
- net PTB0: now reaches U17.8 (PTB0/IRQ_5)
- net PTB1: now reaches U17.9 (PTB1/IRQ_6)
- net CS: now reaches U18.1 (/CS)
- net D1: now reaches U18.2 (DO(IO1))
- net D2: now reaches U18.3 (/WP(IO2))
- net D0: now reaches U18.5 (DI(IO0))
- net CLK: now reaches U18.6 (CLK)
- net D3: now reaches U18.7 (/HOLD_/RESET)
- new net: D22.1 (K), R32.1

Commit message: 12-March update
Changed lines of the file:
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@@
+		(color 0 0 0 0)
+	)
+	(junction
+		(at 226.06 72.39)
+		(diameter 0)
 		(color 0 0 0 0)
 	)
@@
 		)
 		(stroke
+			(width 0)
+			(type default)
+		)
+	)
+	(wire
+		(pts
+			(xy 226.06 71.12) (xy 226.06 72.39)
+		)
+		(stroke

Commit message: test gpg
Parts:
- removed D14, D15: BZV55B5V1, Diode_SMD:D_MiniMELF, symbol Diode:BZV55B5V1
- PROG1: footprint Resistor_SMD:R_0402_1005Metric_Pad0.72x0.64mm_HandSolder -> Resistor_SMD:R_2010_5025Metric_Pad1.40x2.65mm_HandSolder; now not fitted
Connections:
- net MPU-D+: now also J6.A6 (D+), J6.B6 (D+)
- net MPU-D-: now also J6.A7 (D-), J6.B7 (D-)
Changed lines of the file:
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@@
+	)
+	(junction
+		(at 248.92 53.34)
+		(diameter 0)
+		(color 0 0 0 0)
 	)
 	(junction
@@
 	)
 	(junction
-		(at 248.92 53.34)
-		(diameter 0)
-		(color 0 0 0 0)
-	)
-	(junction
 		(at 226.06 72.39)
 		(diameter 0)
@@
 	(wire
 		(pts
-			(xy 248.92 48.26) (xy 248.92 49.53)
+			(xy 248.92 46.99) (xy 248.92 48.26)
 		)
 		(stroke
@@
 	(wire
 		(pts
-			(xy 257.81 142.24) (xy 257.81 143.51)
+			(xy 248.92 48.26) (xy 256.54 48.26)
 		)
 		(stroke
@@
 	(wire
 		(pts
-			(xy 248.92 52.07) (xy 248.92 53.34)
+			(xy 257.81 142.24) (xy 257.81 143.51)
 		)
 		(stroke
@@
 	(wire
 		(pts
-			(xy 30.48 72.39) (xy 44.45 72.39)
+			(xy 248.92 48.26) (xy 248.92 49.53)
 		)
 		(stroke
@@
 	(wire
 		(pts
-			(xy 248.92 53.34) (xy 248.92 54.61)
+			(xy 248.92 52.07) (xy 248.92 53.34)
 		)
 		(stroke
@@
 	(wire
 		(pts
-			(xy 248.92 46.99) (xy 248.92 48.26)
+			(xy 248.92 53.34) (xy 256.54 53.34)
+		)
+		(stroke
+			(width 0)
+			(type default)
+		)
+	)
+	(wire
+		(pts
+			(xy 30.48 72.39) (xy 44.45 72.39)
+		)
+		(stroke
+			(width 0)
+			(type default)
+		)
+	)
+	(wire
+		(pts
+			(xy 248.92 53.34) (xy 248.92 54.61)
 		)
 		(stroke
@@
 			)
 		)
+		(property "KLC_S4.2_DVDD" ""
+			(at 252.73 41.91 90)
+			(effects
+				(font
+					(size 1.27 1.27)
+				)
+				(hide yes)
+			)
+		)
+		(property "KLC_S4.2_VREG_LX" ""
+			(at 252.73 41.91 90)
+			(effects
+				(font
+					(size 1.27 1.27)
+				)
+				(hide yes)
+			)
+		)
 		(pin "1"
 		)
@@
 				(path "/e8b263af-d576-40b7-a774-1c6d96794e54/5ef537cb-0f63-4925-9030-5c1558b6d930"
 					(reference "#PWR099")
-					(unit 1)
-				)
-			)
-		)
-	)
-	(symbol
-		(lib_id "Diode:BZV55B5V1")
-		(at 252.73 48.26 180)
-		(unit 1)
-		(exclude_from_sim no)
-		(in_bom yes)
-		(on_board yes)
-		(dnp no)
-		(property "Reference" "D14"
-			(at 254.508 46.482 0)
-			(effects
-				(font
-					(size 1.27 1.27)
-				)
-			)
-		)
-		(property "Value" "BZV55B5V1"
-			(at 252.73 44.45 0)
-			(effects
-				(font
-					(size 1.27 1.27)
-				)
-			)
-		)
-		(property "Footprint" "Diode_SMD:D_MiniMELF"
-			(at 252.73 43.815 0)
-			(effects
-				(font
-					(size 1.27 1.27)
-				)
-				(hide yes)
-			)
-		)
-		(property "Datasheet" "https://assets.nexperia.com/documents/data-sheet/BZV55_SER.pdf"
-			(at 252.73 48.26 0)
-			(effects
-				(font
-					(size 1.27 1.27)
-				)
-				(hide yes)
-			)
-		)
-		(property "Description" "5.1V, 500mW, 2%, Zener diode, MiniMELF"
-			(at 252.73 48.26 0)
-			(effects
-				(font
-					(size 1.27 1.27)
-				)
-				(hide yes)
-			)
-		)
-		(pin "1"
-		)
-		(pin "2"
-		)
-		(instances
-			(project "Blitz"
-				(path "/e8b263af-d576-40b7-a774-1c6d96794e54/5ef537cb-0f63-4925-9030-5c1558b6d930"
-					(reference "D14")
 					(unit 1)
 				)
@@
 			)
 		)
+		(property "KLC_S4.2_DVDD" ""
+			(at 77.47 80.01 0)
+			(effects
+				(font
+					(size 1.27 1.27)
+				)
+				(hide yes)
+			)
+		)
+		(property "KLC_S4.2_VREG_LX" ""
+			(at 77.47 80.01 0)
+			(effects
+				(font
+					(size 1.27 1.27)
+				)
+				(hide yes)
+			)
+		)
 		(pin "5"
 		)
@@
 			)
 		)
+		(property "KLC_S4.2_DVDD" ""
+			(at 26.67 72.39 90)
+			(effects
+				(font
+					(size 1.27 1.27)
+				)
+				(hide yes)
+			)
+		)
+		(property "KLC_S4.2_VREG_LX" ""
+			(at 26.67 72.39 90)
+			(effects
+				(font
+					(size 1.27 1.27)
+				)
+				(hide yes)
+			)
+		)
 		(pin "1"
 		)
@@
 			)
 		)
+		(property "KLC_S4.2_DVDD" ""
+			(at 233.68 49.53 0)
+			(effects
+				(font
+					(size 1.27 1.27)
+				)
+				(hide yes)
+			)
+		)
+		(property "KLC_S4.2_VREG_LX" ""
+			(at 233.68 49.53 0)
+			(effects
+				(font
+					(size 1.27 1.27)
+				)
+				(hide yes)
+			)
+		)
 		(pin "A5"
 		)
@@
 		(in_bom yes)
 		(on_board yes)
-		(dnp no)
+		(dnp yes)
 		(property "Reference" "PROG1"
 			(at 120.65 68.072 90)
@@
 			)
 		)
-		(property "Footprint" "Resistor_SMD:R_0402_1005Metric_Pad0.72x0.64mm_HandSolder"
+		(property "Footprint" "Resistor_SMD:R_2010_5025Metric_Pad1.40x2.65mm_HandSolder"
 			(at 114.3 71.628 90)
 			(effects
@@
 		(property "Description" "Resistor"
 			(at 114.3 69.85 0)
+			(effects
+				(font
+					(size 1.27 1.27)
+				)
+				(hide yes)
+			)
+		)
+		(property "KLC_S4.2_DVDD" ""
+			(at 114.3 69.85 90)
+			(effects
+				(font
+					(size 1.27 1.27)
+				)
+				(hide yes)
+			)
+		)
+		(property "KLC_S4.2_VREG_LX" ""
+			(at 114.3 69.85 90)
 			(effects
 				(font
@@
 			)
 		)
+		(property "KLC_S4.2_DVDD" ""
+			(at 173.99 143.51 0)
+			(effects
+				(font
+					(size 1.27 1.27)
+				)
+				(hide yes)
+			)
+		)
+		(property "KLC_S4.2_VREG_LX" ""
+			(at 173.99 143.51 0)
+			(effects
+				(font
+					(size 1.27 1.27)
+				)
+				(hide yes)
+			)
+		)
 		(pin "1"
 		)
@@
 		)
 		(property "Sim.Pins" "1=K 2=A"
+			(at 266.7 143.51 0)
+			(effects
+				(font
+					(size 1.27 1.27)
+				)
+				(hide yes)
+			)
+		)
+		(property "KLC_S4.2_DVDD" ""
+			(at 266.7 143.51 0)
+			(effects
+				(font
+					(size 1.27 1.27)
+				)
+				(hide yes)
+			)
+		)
+		(property "KLC_S4.2_VREG_LX" ""
 			(at 266.7 143.51 0)
 			(effects
@@
 			)
 		)
+		(property "KLC_S4.2_DVDD" ""
+			(at 252.73 39.37 90)
+			(effects
+				(font
+					(size 1.27 1.27)
+				)
+				(hide yes)
+			)
+		)
+		(property "KLC_S4.2_VREG_LX" ""
+			(at 252.73 39.37 90)
+			(effects
+				(font
+					(size 1.27 1.27)
+				)
+				(hide yes)
+			)
+		)
 		(pin "1"
 		)
@@
 				(path "/e8b263af-d576-40b7-a774-1c6d96794e54/5ef537cb-0f63-4925-9030-5c1558b6d930"
 					(reference "R22")
-					(unit 1)
-				)
-			)
-		)
-	)
-	(symbol
-		(lib_id "Diode:BZV55B5V1")
-		(at 252.73 53.34 180)
-		(unit 1)
-		(exclude_from_sim no)
-		(in_bom yes)
-		(on_board yes)
-		(dnp no)
-		(fields_autoplaced yes)
-		(property "Reference" "D15"
-			(at 252.73 46.99 0)
-			(effects
-				(font
-					(size 1.27 1.27)
-				)
-			)
-		)
-		(property "Value" "BZV55B5V1"
-			(at 252.73 49.53 0)
-			(effects
-				(font
-					(size 1.27 1.27)
-				)
-			)
-		)
-		(property "Footprint" "Diode_SMD:D_MiniMELF"
-			(at 252.73 48.895 0)
-			(effects
-				(font
-					(size 1.27 1.27)
-				)
-				(hide yes)
-			)
-		)
-		(property "Datasheet" "https://assets.nexperia.com/documents/data-sheet/BZV55_SER.pdf"
-			(at 252.73 53.34 0)
-			(effects
-				(font
-					(size 1.27 1.27)
-				)
-				(hide yes)
-			)
-		)
-		(property "Description" "5.1V, 500mW, 2%, Zener diode, MiniMELF"
-			(at 252.73 53.34 0)
-			(effects
-				(font
-					(size 1.27 1.27)
-				)
-				(hide yes)
-			)
-		)
-		(pin "1"
-		)
-		(pin "2"
-		)
-		(instances
-			(project "Blitz"
-				(path "/e8b263af-d576-40b7-a774-1c6d96794e54/5ef537cb-0f63-4925-9030-5c1558b6d930"
-					(reference "D15")
 					(unit 1)
 				)
@@
 			)
 		)
+		(property "KLC_S4.2_DVDD" ""
+			(at 252.73 34.29 0)
+			(effects
+				(font
+					(size 1.27 1.27)
+				)
+				(hide yes)
+			)
+		)
+		(property "KLC_S4.2_VREG_LX" ""
+			(at 252.73 34.29 0)
+			(effects
+				(font
+					(size 1.27 1.27)
+				)
+				(hide yes)
+			)
+		)
 		(pin "1"
 		)
@@
 			(effects
 				(font
+					(size 1.27 1.27)
+				)
+				(hide yes)
+			)
+		)
+		(property "KLC_S4.2_DVDD" ""
+			(at 274.32 143.51 90)
+			(effects
+				(font
+					(size 1.27 1.27)
+				)
+				(hide yes)
+			)
+		)
+		(property "KLC_S4.2_VREG_LX" ""
+			(at 274.32 143.51 90)
+			(effects
+				(font
