File: Hardware/Navigation.kicad_sch (KiCad schematic)
At the start: 42 parts, among them J1 USB_C_Receptacle_USB2.0_16P, J2 SM03B-SRSS-TB_LF__SN_, U1 RP2350B, U10 W25Q128JVS, U11 W25Q128JVS, U3 AP2112K-3.3, Y1 ABM8-272-T3

Commit message: 27 feb update
Parts:
- removed U3: AP2112K-3.3, Package_TO_SOT_SMD:SOT-23-5, symbol Regulator_Linear:AP2112K-3.3
- added C48: 10uF, Capacitor_SMD:C_1206_3216Metric_Pad1.33x1.80mm_HandSolder, symbol Device:C
- added C49: 22uF, Capacitor_SMD:C_1206_3216Metric_Pad1.33x1.80mm_HandSolder, symbol Device:C
- added C53, C54: 1uF, Capacitor_SMD:C_1206_3216Metric_Pad1.33x1.80mm_HandSolder, symbol Device:C
- added D16, D17: BZV55B5V1, Diode_SMD:D_MiniMELF, symbol Diode:BZV55B5V1
- added R30: 64, Resistor_SMD:R_0201_0603Metric, symbol Device:R
- added U20: TLV75733PDRV, Package_SON:WSON-6-1EP_2x2mm_P0.65mm_EP1x1.6mm, symbol Regulator_Linear:TLV75733PDRV
- added U3: TPS2113ADRBR, TPS2113ADRBR:SON65P300X300X100-9N, symbol TPS2113ADRBR:TPS2113ADRBR
- R19, R4: value DNF -> DNP
Connections:
- net +5V: now also D17.2 (A)
- net GND: now also U1.81 (GND), C48.2, C49.2, C53.2, C54.1, R30.2, U20.3 (GND), U20.7 (GND), U3.5 (GND), U3.9 (GND)
- net Nav-3.3V: now also C54.2, U20.1 (OUT)
- net Nav-5V: now also D16.2 (A)
- net at D5.1 (K): now also C49.1, U3.6 (IN2); no longer D4.1 (K)
- new net: D16.1 (K), D17.1 (K), U3.2 (~{EN})
- new net: R30.1, U3.4 (ILIM)
- new net: C53.1, U20.4 (EN), U20.6 (IN), U3.7 (OUT)
- new net: C48.1, D4.1 (K), U3.8 (IN1)
Other:
- moved on the sheet: J2

Commit message: 12-March update
Parts:
- removed C16: 100nF, Capacitor_SMD:C_01005_0402Metric, symbol Device:C
- removed C53, C54: 1uF, Capacitor_SMD:C_1206_3216Metric_Pad1.33x1.80mm_HandSolder, symbol Device:C
- removed D1, D2: BZV55B5V1, Diode_SMD:D_MiniMELF, symbol Diode:BZV55B5V1
- removed L1: 3.3u, Capacitor_SMD:C_0201_0603Metric, symbol Device:L
- removed R19, R4: DNP, Resistor_SMD:R_0603_1608Metric, symbol Device:R
- removed U10: W25Q128JVS, Package_SO:SOIC-8_5.3x5.3mm_P1.27mm, symbol Memory_Flash:W25Q128JVS
- added C37, C41: 1uF, Capacitor_SMD:C_0402_1005Metric, symbol Device:C
- added D1, D30: 1N4148WT, Diode_SMD:D_SOD-523, symbol Diode:1N4148WT
- added D2: WS2812, LED_SMD:LED_WS2812_PLCC6_5.0x5.0mm_P1.6mm, symbol LED:WS2812
- added D26, D27: 1N914WT, Diode_SMD:D_SOD-523, symbol Diode:1N914WT
- added DNP1, DNP2: R, Resistor_SMD:R_2010_5025Metric_Pad1.40x2.65mm_HandSolder, symbol Device:R
- added L3: AOTA-B201610S3R3-101-T, AOTAB201610S3R3101T, symbol AOTA-B201610S3R3-101-T:AOTA-B201610S3R3-101-T
- added Q3: 2N7002, Package_TO_SOT_SMD:SOT-23, symbol Transistor_FET:2N7002
- added R26, R31: 4.7K, Resistor_SMD:R_0201_0603Metric, symbol Device:R
Connections:
- net GND: now also C37.2, C41.2, D2.3 (VCC), D2.6 (VSS), Q3.2 (S)
- net Nav-3.3V: now also C37.1, L3.2, R26.2, R31.1
- net Nav-D+: now also D1.1 (K)
- net Nav-D-: now also D30.1 (K)
- net Nav-GPIO0: no longer U11.1 (~{CS})
- net Nav-QSPI_SS: now also U11.1 (~{CS}), DNP1.1
- net Nav-RUN: now also D26.2 (A)
- net at J1.A6 (D+), J1.B6 (D+): now also D1.2 (A)
- net NAV-SDA: now reaches U1.1 (GPIO4)
- net NAV-SDA: now also R26.1
- net NAV-MPU-MISO: now reaches U1.11 (GPIO12)
- net NAV-MPU-CS: now reaches U1.12 (GPIO13)
- net NAV-TEL-SDA: now reaches U1.13 (GPIO14)
- net NAV-TEL-SCL: now reaches U1.14 (GPIO15)
- net NAV-MISO: now reaches U1.16 (GPIO16)
- net NAV-SCK: now reaches U1.18 (GPIO18)
- net NAV-MOSI: now reaches U1.19 (GPIO19)
- net NAV-SCL: now reaches U1.2 (GPIO5)
- net NAV-SCL: now also R31.2
- net BMI088-INT-3: now reaches U1.20 (GPIO20)
- net BMI088-INT-4: now reaches U1.21 (GPIO21)
- net BMM350-INT: now reaches U1.22 (GPIO22)
- net BMP581-INT: now reaches U1.23 (GPIO23)
- net Nav-stat: now reaches U1.3 (GPIO6)
- net Nav-stat: now also D2.2 (DIN)
- net NAV-GYRO-CS: now reaches U1.42 (GPIO33)
- net NAV-ACC-CS: now reaches U1.46 (GPIO37)
- net NAV-RADIO-CS: now reaches U1.52 (GPIO41/ADC1)
- net BMI088-INT-1: now reaches U1.6 (GPIO8)
- net at U1.63 (VREG_LX): now also L3.1
- net BMI088-INT-2: now reaches U1.7 (GPIO9)
- net GPS-RESET: now reaches U1.78 (GPIO1)
- net Timepulse: now reaches U1.79 (GPIO2)
- net NAV-MPU-SCK: now reaches U1.8 (GPIO10)
- net RTC-1MHZ: now reaches U1.80 (GPIO3)
- net NAV-MPU-MOSI: now reaches U1.9 (GPIO11)
- net Nav-5V-stable: now reaches U20.4 (EN), U20.6 (IN), U3.7 (OUT)
- net Nav-5V-stable: now also C41.1, D2.5 (VDD)
- net at R5.1: now also DNP1.2
- net at J1.A7 (D-), J1.B7 (D-): now also D30.2 (A)
- net at R20.1: now also DNP2.2
- new net: D27.2 (A), Q3.3 (D)
- new net: D26.1 (K), D27.1 (K), DNP2.1
- new net Nav-RESET: Q3.1 (G)
Other:
- moved on the sheet: C18, C19, R6, Y1

Commit message: test gpg
Parts:
- removed D1, D30: 1N4148WT, Diode_SMD:D_SOD-523, symbol Diode:1N4148WT
- DNP1, DNP2: now not fitted
Connections:
- net Nav-D+: now also J1.A6 (D+), J1.B6 (D+)
- net Nav-D-: now also J1.A7 (D-), J1.B7 (D-)
