File: Hardware/Power.kicad_sch (KiCad schematic)
At the start: 11 parts, among them U7 SY8205FCC, U8 AP2112K-3.3, U9 AP2112K-1.8

Commit message: 27 feb update
Parts:
- removed U8: AP2112K-3.3, Package_TO_SOT_SMD:SOT-23-5, symbol Regulator_Linear:AP2112K-3.3
- added C43, C50: 1uF, Capacitor_SMD:C_1206_3216Metric_Pad1.33x1.80mm_HandSolder, symbol Device:C
- added U22: TLV75733PDRV, Package_SON:WSON-6-1EP_2x2mm_P0.65mm_EP1x1.6mm, symbol Regulator_Linear:TLV75733PDRV
Connections:
- net +3.3V: now also C50.2, U22.1 (OUT)
- net +5V: now also C43.1, U22.4 (EN), U22.6 (IN)
- net GND: now also C43.2, C50.1, U22.3 (GND), U22.7 (GND)

Commit message: 12-March update
Parts:
- removed C37: 100nf, Capacitor_SMD:C_1206_3216Metric_Pad1.33x1.80mm_HandSolder, symbol Device:C
- removed C39: 1uf, Capacitor_SMD:C_1206_3216Metric_Pad1.33x1.80mm_HandSolder, symbol Device:C
- removed C40: 10uf, Capacitor_SMD:C_0402_1005Metric, symbol Device:C
- removed C41: C_Polarized_Small, Capacitor_SMD:CP_Elec_3x5.3, symbol Device:C_Polarized_Small
- removed L3: 3.3uH-XAL7030-332ME, Inductor_SMD:L_6.3x6.3_H3, symbol Device:L
- added C51: 50nF, Capacitor_SMD:C_0201_0603Metric, symbol Device:C
- added H1, H2: Batsolderpad, TestPoint:TestPoint_Pad_4.0x4.0mm, symbol Mechanical:Batsolderpad
- added L2: SPM4012T-2R2M, SPM4012T-2R2M:IND_SPM4012T-2R2M, symbol SPM4012T-2R2M:SPM4012T-2R2M
- C42: value 100nf -> C; footprint Capacitor_SMD:C_0402_1005Metric -> (none)
- R23: value 110k -> 44.2k; footprint Resistor_SMD:R_0508_1220Metric_Pad1.12x2.15mm_HandSolder -> Resistor_SMD:R_0402_1005Metric
- R24: value 15k -> 6.04k; footprint Resistor_SMD:R_0508_1220Metric -> Resistor_SMD:R_0402_1005Metric
Connections:
- net +5V: now also R23.2, L2.2; no longer R23.1
- net GND: now also R24.2, C51.1, H2.1; no longer C42.1, R24.1
- net at C42.2: now also U7.2 (LX), L2.1; no longer U7.4 (SS)
- net at U7.1 (BS): now also C42.1
- net PVIN renamed +24V
- net +24V: now also H1.1
- new net: R23.1, R24.1, U7.5 (FB)
- new net: C51.2, U7.4 (SS)

Commit message: test gpg
Parts:
- removed C42: C, symbol Device:C
- removed C51: 50nF, Capacitor_SMD:C_0201_0603Metric, symbol Device:C
- removed L2: SPM4012T-2R2M, SPM4012T-2R2M:IND_SPM4012T-2R2M, symbol SPM4012T-2R2M:SPM4012T-2R2M
- removed R23: 44.2k, Resistor_SMD:R_0402_1005Metric, symbol Device:R
- removed R24: 6.04k, Resistor_SMD:R_0402_1005Metric, symbol Device:R
- removed U7: SY8205FCC, SY8205FCC:VREG_SY8205FCC, symbol SY8205FCC:SY8205FCC
- added U15: TPS54302, Package_TO_SOT_SMD:SOT-23-6, symbol Regulator_Switching:TPS54302
