File: Hardware/Telemetry.kicad_sch (KiCad schematic)
At the start: 41 parts, among them J3 Micro_SD_Card_Det2, J4 SM03B-SRSS-TB_LF__SN_, J5 USB_C_Receptacle_USB2.0_16P, U12 RP2350B, U13 AP2112K-3.3, U15 W25Q128JVS, Y2 ABM8-272-T3

Commit message: 27 feb update
Parts:
- removed R13, R17: DNF, Resistor_SMD:R_0603_1608Metric, symbol Device:R
- removed U13: AP2112K-3.3, Package_TO_SOT_SMD:SOT-23-5, symbol Regulator_Linear:AP2112K-3.3
- added C46: 10uF, Capacitor_SMD:C_1206_3216Metric_Pad1.33x1.80mm_HandSolder, symbol Device:C
- added C47: 22uF, Capacitor_SMD:C_1206_3216Metric_Pad1.33x1.80mm_HandSolder, symbol Device:C
- added C51, C52: 1uF, Capacitor_SMD:C_1206_3216Metric_Pad1.33x1.80mm_HandSolder, symbol Device:C
- added D18, D19: BZV55B5V1, Diode_SMD:D_MiniMELF, symbol Diode:BZV55B5V1
- added R29: 64, Resistor_SMD:R_0201_0603Metric, symbol Device:R
- added U13: TPS2113ADRBR, TPS2113ADRBR:SON65P300X300X100-9N, symbol TPS2113ADRBR:TPS2113ADRBR
- added U19: TLV75733PDRV, Package_SON:WSON-6-1EP_2x2mm_P0.65mm_EP1x1.6mm, symbol Regulator_Linear:TLV75733PDRV
Connections:
- net +5V: now also D18.2 (A)
- net GND: now also J3.11 (SHIELD), J3.6 (VSS), U12.81 (GND), C46.2, C47.2, C51.2, C52.1, R29.2, U13.5 (GND), U13.9 (GND), U19.3 (GND), U19.7 (GND)
- net Tel-3.3V: now also J3.4 (VDD), C52.2, U19.1 (OUT)
- net Tel-5V: now also D19.2 (A)
- net at D6.1 (K): now also C46.1, U13.8 (IN1); no longer D7.1 (K)
- net TEL-DET: now reaches U12.14 (GPIO15)
- net TEL-DET: now also J3.10 (DET_A), J3.9 (DET_B)
- net TEL-MISO: now reaches U12.16 (GPIO16)
- net TEL-MISO: now also J3.7 (DAT0)
- net TEL-CS: now reaches U12.17 (GPIO17)
- net TEL-CS: now also J3.2 (DAT3/CD)
- net TEL-SCK: now reaches U12.18 (GPIO18)
- net TEL-SCK: now also J3.5 (CLK)
- net TEL-MOSI: now reaches U12.19 (GPIO19)
- net TEL-MOSI: now also J3.3 (CMD)
- new net: D18.1 (K), D19.1 (K), U13.2 (~{EN})
- new net: C51.1, U13.7 (OUT), U19.4 (EN), U19.6 (IN)
- new net: C47.1, D7.1 (K), U13.6 (IN2)
- new net: R29.1, U13.4 (ILIM)
Other:
- moved on the sheet: J4

Commit message: 12-March update
Parts:
- removed C38: 100nF, Capacitor_SMD:C_01005_0402Metric, symbol Device:C
- removed C51, C52: 1uF, Capacitor_SMD:C_1206_3216Metric_Pad1.33x1.80mm_HandSolder, symbol Device:C
- removed L2: 3.3u, Inductor_SMD:L_0201_0603Metric, symbol Device:L
- removed R18: 10, Resistor_SMD:R_0201_0603Metric_Pad0.64x0.40mm_HandSolder, symbol Device:R
- removed U15: W25Q128JVS, Package_SO:SOIC-8_5.3x5.3mm_P1.27mm, symbol Memory_Flash:W25Q128JVS
- added C16: 100nF, Capacitor_SMD:C_01005_0402Metric, symbol Device:C
- added C39, C40: 1uF, Capacitor_SMD:C_0402_1005Metric, symbol Device:C
- added D28, D29: 1N914WT, Diode_SMD:D_SOD-523, symbol Diode:1N914WT
- added D31: WS2812, LED_SMD:LED_WS2812_PLCC6_5.0x5.0mm_P1.6mm, symbol LED:WS2812
- added DNP3, DNP4: R, Resistor_SMD:R_2010_5025Metric_Pad1.40x2.65mm_HandSolder, symbol Device:R
- added L1: AOTA-B201610S3R3-101-T, AOTAB201610S3R3101T, symbol AOTA-B201610S3R3-101-T:AOTA-B201610S3R3-101-T
- added Q4: 2N7002, Package_TO_SOT_SMD:SOT-23, symbol Transistor_FET:2N7002
- added R25, R27: 4.7K, Resistor_SMD:R_0201_0603Metric, symbol Device:R
- added R34: 10, Resistor_SMD:R_0201_0603Metric_Pad0.64x0.40mm_HandSolder, symbol Device:R
- added U10: W25Q128JVS, Package_SO:SOIC-8_5.3x5.3mm_P1.27mm, symbol Memory_Flash:W25Q128JVS
Connections:
- net GND: now also C16.2, C39.2, C40.2, D31.3 (VCC), D31.6 (VSS), Q4.2 (S), R34.2, U10.4 (GND)
- net TEL-DET: now also U12.22 (GPIO22); no longer U12.14 (GPIO15)
- net Tel-1.1V: now also L1.2
- net Tel-3.3V: now also C16.1, C39.1, R25.1, R27.2, U10.8 (VCC)
- net Tel-QSPI_SCLK: now also U10.6 (CLK)
- net Tel-QSPI_SD0: now also U10.5 (DI/IO_{0})
- net Tel-QSPI_SD1: now also U10.2 (DO/IO_{1})
- net Tel-QSPI_SD2: now also U10.3 (~{WP}/IO_{2})
- net Tel-QSPI_SD3: now also U10.7 (~{HOLD}/~{RESET}/IO_{3})
- net Tel-QSPI_SS: now also DNP3.1, U10.1 (~{CS})
- net Tel-RUN: now also D28.2 (A)
- net TEL-MPU-MISO: now reaches U12.11 (GPIO12)
- net TEL-MPU-CS: now reaches U12.12 (GPIO13)
- net NAV-TEL-SDA: now reaches U12.13 (GPIO14)
- net NAV-TEL-SDA: now also R27.1
- net TEL-RADIO-SC: now reaches U12.2 (GPIO5)
- net TEL-INT: now reaches U12.20 (GPIO20)
- net TEL-SDN: now reaches U12.21 (GPIO21)
- net at U12.63 (VREG_LX): now also L1.1
- net RTC-1MHZ: now reaches U12.77 (GPIO0)
- net Tel-stat: now reaches U12.78 (GPIO1)
- net Tel-stat: now also D31.2 (DIN)
- net TEL-MPU-SCK: now reaches U12.8 (GPIO10)
- net TEL-MPU-MOSI: now reaches U12.9 (GPIO11)
- net Tel-5V-stable: now reaches U13.7 (OUT), U19.4 (EN), U19.6 (IN)
- net Tel-5V-stable: now also C40.1, D31.5 (VDD)
- net at R14.1: now also DNP3.2
- new net: D28.1 (K), D29.1 (K), DNP4.1
- new net: DNP4.2, R34.1
- new net: D29.2 (A), Q4.3 (D)
- new net NAV-TEL-SCL: R25.2, U12.14 (GPIO15)
- new net Tel-RESET: Q4.1 (G)
Other:
- moved on the sheet: J3

Commit message: test gpg
Parts:
- removed D10, D9: BZV55B5V1, Diode_SMD:D_MiniMELF, symbol Diode:BZV55B5V1
- DNP3, DNP4: now not fitted
Connections:
- net Tel-D+: now also J5.A6 (D+), J5.B6 (D+)
- net Tel-D-: now also J5.A7 (D-), J5.B7 (D-)
