File: Hardware/Programmer.kicad_sch (KiCad schematic)
At the start: 1 part, among them J8 Bus_PCI_Express_x4

Commit message: 12-March update
Parts:
- removed J8: Bus_PCI_Express_x4, Connector_PCBEdge:BUS_PCIexpress_x4, symbol Connector:Bus_PCI_Express_x4
Changed lines of the file:
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@@
 		(date "2026-02-19")
 	)
-	(symbol
-		(lib_id "Connector:Bus_PCI_Express_x4")
-		(at 251.46 78.74 0)
-		(unit 1)
-		(exclude_from_sim no)
-		(in_bom yes)
-		(on_board yes)
-		(dnp no)
-		(fields_autoplaced yes)
-		(property "Reference" "J8"
-			(at 253.6033 110.49 0)
-			(effects
-				(font
-					(size 1.27 1.27)
-				)
-				(justify left)
-			)
-		)
-		(property "Value" "Bus_PCI_Express_x4"
-			(at 253.6033 113.03 0)
-			(effects
-				(font
-					(size 1.27 1.27)
-				)
-				(justify left)
-			)
-		)
-		(property "Footprint" "Connector_PCBEdge:BUS_PCIexpress_x4"
-			(at 251.46 81.28 0)
-			(effects
-				(font
-					(size 1.27 1.27)
-				)
-				(hide yes)
-			)
-		)
-		(property "Datasheet" "http://www.ritrontek.com/uploadfile/2016/1026/20161026105231124.pdf#page=63"
-			(at 245.11 110.49 0)
-			(effects
-				(font
-					(size 1.27 1.27)
-				)
-				(hide yes)
-			)
-		)
-		(property "Description" "PCI Express bus connector x4"
-			(at 251.46 78.74 0)
-			(effects
-				(font
-					(size 1.27 1.27)
-				)
-				(hide yes)
-			)
-		)
-		(pin "A30"
-		)
-		(pin "A29"
-		)
-		(pin "B22"
-		)
-		(pin "B21"
-		)
-		(pin "B18"
-		)
-		(pin "B16"
-		)
-		(pin "B13"
-		)
-		(pin "A4"
-		)
-		(pin "A31"
-		)
-		(pin "A28"
-		)
-		(pin "A27"
-		)
-		(pin "A24"
-		)
-		(pin "A23"
-		)
-		(pin "A20"
-		)
-		(pin "A15"
-		)
-		(pin "A18"
-		)
-		(pin "B2"
-		)
-		(pin "A3"
-		)
-		(pin "B10"
-		)
-		(pin "B3"
-		)
-		(pin "B1"
-		)
-		(pin "A2"
-		)
-		(pin "A12"
-		)
-		(pin "B25"
-		)
-		(pin "B26"
-		)
-		(pin "B29"
-		)
-		(pin "B32"
-		)
-		(pin "B4"
-		)
-		(pin "B7"
-		)
-		(pin "A10"
-		)
-		(pin "A9"
-		)
-		(pin "B8"
-		)
-		(pin "B30"
-		)
-		(pin "A32"
-		)
-		(pin "A19"
-		)
-		(pin "B12"
-		)
-		(pin "B11"
-		)
-		(pin "A11"
-		)
-		(pin "B9"
-		)
-		(pin "A5"
-		)
-		(pin "A6"
-		)
-		(pin "A7"
-		)
-		(pin "A8"
-		)
-		(pin "A16"
-		)
-		(pin "A17"
-		)
-		(pin "A21"
-		)
-		(pin "A22"
-		)
-		(pin "B14"
-		)
-		(pin "B20"
-		)
-		(pin "B27"
-		)
-		(pin "B24"
-		)
-		(pin "B15"
-		)
-		(pin "B23"
-		)
-		(pin "B19"
-		)
-		(pin "B31"
-		)
-		(pin "B17"
-		)
-		(pin "A1"
-		)
-		(pin "A14"
-		)
-		(pin "A13"
-		)
-		(pin "B6"
-		)
-		(pin "B5"
-		)
-		(pin "B28"
-		)
-		(pin "A25"
-		)
-		(pin "A26"
-		)
-		(instances
-			(project ""
-				(path "/e8b263af-d576-40b7-a774-1c6d96794e54/b1b7e2f6-54c8-4556-8c77-aada4a0b3b7d"
-					(reference "J8")
-					(unit 1)
-				)
-			)
-		)
-	)
 )

Commit message: test gpg
Parts:
- added TR2: ADT1-1WT, RF_Mini-Circuits:Mini-Circuits_CD542_H2.84mm, symbol Transformer:ADT1-1WT
Changed lines of the file:
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@@
 		(date "2026-02-19")
 	)
+	(symbol
+		(lib_id "Transformer:ADT1-1WT")
+		(at 100.33 88.9 0)
+		(unit 1)
+		(exclude_from_sim no)
+		(in_bom yes)
+		(on_board yes)
+		(dnp no)
+		(fields_autoplaced yes)
+		(property "Reference" "TR2"
+			(at 100.33 78.74 0)
+			(effects
+				(font
+					(size 1.27 1.27)
+				)
+			)
+		)
+		(property "Value" "ADT1-1WT"
+			(at 100.33 81.28 0)
+			(effects
+				(font
+					(size 1.27 1.27)
+				)
+			)
+		)
+		(property "Footprint" "RF_Mini-Circuits:Mini-Circuits_CD542_H2.84mm"
+			(at 100.33 97.79 0)
+			(effects
+				(font
+					(size 1.27 1.27)
+				)
+				(hide yes)
+			)
+		)
+		(property "Datasheet" "https://www.minicircuits.com/pdfs/ADT1-1WT.pdf"
+			(at 100.33 88.9 0)
+			(effects
+				(font
+					(size 1.27 1.27)
+				)
+				(hide yes)
+			)
+		)
+		(property "Description" "0.005-125MHz 1:1 RF Transformer, Unbalanced to Balanced Center Tap, CD542"
+			(at 100.33 88.9 0)
+			(effects
+				(font
+					(size 1.27 1.27)
+				)
+				(hide yes)
+			)
+		)
+		(pin "6"
+		)
+		(pin "2"
+		)
+		(pin "4"
+		)
+		(pin "1"
+		)
+		(pin "3"
+		)
+		(pin "5"
+		)
+		(instances
+			(project ""
+				(path "/e8b263af-d576-40b7-a774-1c6d96794e54/b1b7e2f6-54c8-4556-8c77-aada4a0b3b7d"
+					(reference "TR2")
+					(unit 1)
+				)
+			)
+		)
+	)
 )
